Commit message: Initial update

File: urdf/nico_grasper.urdf (robot description, URDF)
Before this commit: robot nico_upper_rh6d, 29 links, 28 joints
Links:
- link sight: geometry visual cylinder length=0.6 radius=0.001
Joints:
- removed joint l_litlefinger_x
- removed joint r_litlefinger_x
- added joint l_littlefinger_x: type revolute, parent left_palm, child l_littlefinger, origin xyz=0.00 0.02 -0.06 rpy=0 0 0, axis 0 1 0, limit lower=-2.57 upper=0 effort=30 velocity=1
- added joint r_littlefinger_x: type revolute, parent right_palm, child r_littlefinger, origin xyz=0.00 0.02 -0.06 rpy=0 0 0, axis 0 1 0, limit lower=-2.57 upper=0 effort=30 velocity=1
- joint eyesight: origin xyz=0 0.0 0.0 rpy=0 0 0 -> xyz=0.1 0.0 0.095 rpy=0 0 0
